File: amiga_joyboard.kicad_sch (KiCad schematic)
At the start: 18 parts, among them J1 JOYPORT_OUT, SW1 FIRE_BTN, SW2 B_BTN, SW3 A_BTN, SW4 RIGHT_BTN, SW5 LEFT_BTN, SW6 DOWN_BTN, SW7 UP_BTN, SW8 AUTOFIRE_SW, SW9 AMIGA_C64_SW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

Commit message: boards separated
Parts:
- added J2: CONN_D, Connector_JST:JST_XH_S5B-XH-A_1x05_P2.50mm_Horizontal, symbol Connector:Conn_01x05_Pin
- added J3: CONN_F, Connector_JST:JST_XH_S5B-XH-A_1x05_P2.50mm_Horizontal, symbol Connector:Conn_01x05_Pin
Connections:
- net A renamed A_D
- net A_D: now also J2.3 (Pin_3); no longer SW3.1
- net B renamed B_D
- net B_D: now also J2.2 (Pin_2); no longer SW2.1
- net FIRE renamed FIRE_D
- net FIRE_D: now also J2.1 (Pin_1); no longer SW1.1
- net GND renamed GND_D
- net GND_D: now also J2.5 (Pin_5); no longer C1.2, C2.2, SW8.2 (C), SW9.2 (C), U1.1 (GND)
- net VCC renamed VCC_F
- net VCC_F: now also J3.4 (Pin_4); no longer J1.7
- new net A_F: J3.3 (Pin_3), SW3.1
- new net B_F: J3.2 (Pin_2), SW2.1
- new net FIRE_F: J3.1 (Pin_1), SW1.1
- new net GND_F: C1.2, C2.2, J3.5 (Pin_5), SW8.2 (C), SW9.2 (C), U1.1 (GND)
- new net VCC_D: J1.7, J2.4 (Pin_4)
Other:
- moved on the sheet: J1, SW4, SW5, SW6, SW7

Commit message: first complete design
Parts:
- R1: value 270 -> 100
Changed lines of the file:
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@@
 			)
 		)
-		(property "Value" "270"
+		(property "Value" "100"
 			(at 120.65 142.24 90)
 			(effects

Commit message: footprints cleanup - kailh copied to local footprints dir
Parts:
- SW1, SW2, SW3, SW4, SW5, SW6, SW7: footprint Kailh:SW_MX -> Amiga Joyboard:SW_MX
Changed lines of the file:
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@@
 			)
 		)
-		(property "Footprint" "Kailh:SW_MX"
+		(property "Footprint" "Amiga Joyboard:SW_MX"
 			(at 91.44 59.69 0)
 			(effects
@@
 			)
 		)
-		(property "Footprint" "Kailh:SW_MX"
+		(property "Footprint" "Amiga Joyboard:SW_MX"
 			(at 91.44 49.53 0)
 			(effects
@@
 			)
 		)
-		(property "Footprint" "Kailh:SW_MX"
+		(property "Footprint" "Amiga Joyboard:SW_MX"
 			(at 85.09 146.05 0)
 			(effects
@@
 			)
 		)
-		(property "Footprint" "Kailh:SW_MX"
+		(property "Footprint" "Amiga Joyboard:SW_MX"
 			(at 91.44 29.21 0)
 			(effects
@@
 			)
 		)
-		(property "Footprint" "Kailh:SW_MX"
+		(property "Footprint" "Amiga Joyboard:SW_MX"
 			(at 85.09 135.89 0)
 			(effects
@@
 			)
 		)
-		(property "Footprint" "Kailh:SW_MX"
+		(property "Footprint" "Amiga Joyboard:SW_MX"
 			(at 91.44 39.37 0)
 			(effects
@@
 			)
 		)
-		(property "Footprint" "Kailh:SW_MX"
+		(property "Footprint" "Amiga Joyboard:SW_MX"
 			(at 85.09 120.65 0)
 			(effects
