File: yboard_rounded.kicad_pcb (KiCad board)
At the start: 2 copper layers, 192.5 x 63.5 mm, 29 parts, among them J1 JOYPORT_OUT, J2 CONN_D, J3 CONN_F, SW1 FIRE_BTN, SW2 B_BTN, SW3 A_BTN, SW4 RIGHT_BTN, SW5 LEFT_BTN, SW6 DOWN_BTN, SW7 UP_BTN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

Commit message: YBoard rename within the designs
Other:
- board text added: "YBoard DirBoard v 1.0"
- board text added: "YBoard FireBoard"
- board text removed: "JoyBoard DirBoard v 1.0"
- board text removed: "JoyBoard FireBoard"
