File: yboard.kicad_sch (KiCad schematic)
At the start: 20 parts, among them J1 JOYPORT_OUT, J2 CONN_D, J3 CONN_F, SW1 FIRE_BTN, SW2 B_BTN, SW3 A_BTN, SW4 RIGHT_BTN, SW5 LEFT_BTN, SW6 DOWN_BTN, SW7 UP_BTN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

Commit message: YBoard rename within the designs
Other:
- title: Amiga JoyBoard -> YBoard
Changed lines of the file:
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@@
 	(paper "A4")
 	(title_block
-		(title "Amiga JoyBoard")
+		(title "YBoard")
 		(date "2024-07-07")
 		(rev "1.0")

Commit message: labeling, libraries and other minor fixes
Parts:
- SW1, SW2, SW3, SW4, SW5, SW6, SW7: footprint Amiga Joyboard:SW_MX -> Yboard:SW_MX
- SW8, SW9: footprint Amiga Joyboard:SS12T44_SLIDER_SWITCH_SPDT -> Yboard:SS12T44_SLIDER_SWITCH_SPDT
Changed lines of the file:
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@@
 			)
 		)
-		(property "Footprint" "Amiga Joyboard:SW_MX"
+		(property "Footprint" "Yboard:SW_MX"
 			(at 91.44 59.69 0)
 			(effects
@@
 			)
 		)
-		(property "Footprint" "Amiga Joyboard:SW_MX"
+		(property "Footprint" "Yboard:SW_MX"
 			(at 91.44 49.53 0)
 			(effects
@@
 			)
 		)
-		(property "Footprint" "Amiga Joyboard:SW_MX"
+		(property "Footprint" "Yboard:SW_MX"
 			(at 85.09 146.05 0)
 			(effects
@@
 			)
 		)
-		(property "Footprint" "Amiga Joyboard:SW_MX"
+		(property "Footprint" "Yboard:SW_MX"
 			(at 91.44 29.21 0)
 			(effects
@@
 			)
 		)
-		(property "Footprint" "Amiga Joyboard:SW_MX"
+		(property "Footprint" "Yboard:SW_MX"
 			(at 85.09 135.89 0)
 			(effects
@@
 			)
 		)
-		(property "Footprint" "Amiga Joyboard:SW_MX"
+		(property "Footprint" "Yboard:SW_MX"
 			(at 91.44 39.37 0)
 			(effects
@@
 			)
 		)
-		(property "Footprint" "Amiga Joyboard:SW_MX"
+		(property "Footprint" "Yboard:SW_MX"
 			(at 85.09 120.65 0)
 			(effects
@@
 			)
 		)
-		(property "Footprint" "Amiga Joyboard:SS12T44_SLIDER_SWITCH_SPDT"
+		(property "Footprint" "Yboard:SS12T44_SLIDER_SWITCH_SPDT"
 			(at 132.08 156.21 0)
 			(effects
@@
 			)
 		)
-		(property "Footprint" "Amiga Joyboard:SS12T44_SLIDER_SWITCH_SPDT"
+		(property "Footprint" "Yboard:SS12T44_SLIDER_SWITCH_SPDT"
 			(at 101.6 135.89 0)
 			(effects
