File: yboard.kicad_pcb (KiCad board)
At the start: 2 copper layers, 192.5 x 63.5 mm, 29 parts, among them J1 JOYPORT_OUT, J2 CONN_D, J3 CONN_F, SW1 AF_SW, SW1 FIRE_BTN, SW2 B_BTN, SW3 A_BTN, SW4 RIGHT_BTN, SW5 LEFT_BTN, SW6 DOWN_BTN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

Commit message: footprint number fix
Parts:
- renumbered SW1 to SW8

Commit message: v number update
Other:
- board text added: "YBoard DirBoard v 1.1"
- board text added: "v 1.1"
- board text removed: "YBoard DirBoard v 1.0"
- board text removed: "v 1.0"
